Commit message: changed to camera observation

File: grasp_gym/environments/models/panda_gripper/gripper_model.urdf (robot description, URDF)
Before this commit: robot panda, 8 links, 7 joints
Links:
- added link camera_lense, mass 0.1; visual cylinder length=0.001 radius=0.005
- added link camera_link, mass 0.1; visual box size=0.02 0.05 0.02
- added link y_rot_link, mass 1.2
- added link z_rot_link, mass 1.2
Joints:
- removed joint panda_hand_joint
- added joint camera_lense_joint: type fixed, parent camera_link, child camera_lense, origin xyz=0 0 0.01 rpy=0 0 0
- added joint camera_mount_joint: type fixed, parent panda_hand, child camera_link, origin xyz=0.03 0 0.05 rpy=0 0 0
- added joint panda_gripper_joint: type fixed, parent y_rot_link, child panda_hand, origin xyz=0 0 0.1 rpy=0 0 0
- added joint panda_rot_y_joint: type revolute, parent z_rot_link, child y_rot_link, origin xyz=0 0 0 rpy=0 0 0, axis 0 1 0, limit lower=-1 upper=1 effort=1 velocity=1
- added joint panda_rot_z_joint: type revolute, parent z_link, child z_rot_link, origin xyz=0 0 0 rpy=3.14159265359 0 0, axis 0 0 1, limit lower=-1 upper=1 effort=1 velocity=1
